Commit message: Update robot.xacro

File: src/my_robot/model/robot.xacro (robot description, xacro)
@@ -1,32 +1,56 @@
 <?xml version="1.0"?>
 <robot xmlns:xacro="http://www.ros.org/wiki/xacro" name="differential_drive_robot">
-  <!-- ═══════════════ XACRO PROPERTIES ═══════════════ -->
-  <xacro:property name="chassis_length"    value="0.20"/>
-  <xacro:property name="chassis_width"     value="0.15"/>
-  <xacro:property name="chassis_height"    value="0.03"/>
-  <xacro:property name="wheel_radius"      value="0.0325"/>
-  <xacro:property name="wheel_width"       value="0.025"/>
-  <xacro:property name="wheel_separation"  value="0.176"/>
-  <xacro:property name="caster_radius"     value="0.012"/>
-  <xacro:property name="chassis_z"         value="${wheel_radius}"/>
-  <xacro:property name="bat_l"    value="0.055"/>
-  <xacro:property name="bat_w"    value="0.030"/>
-  <xacro:property name="bat_h"    value="0.012"/>
-  <xacro:property name="bat_gap"  value="0.005"/>
-  <xacro:property name="bat_pitch" value="${bat_w + bat_gap}"/>
+  <!-- ════════════════════════════════════════════════════════
+       XACRO PROPERTIES
+       ════════════════════════════════════════════════════════ -->
+  <!-- Chassis dimensions -->
+  <xacro:property name="chassis_length"   value="0.20"/>
+  <xacro:property name="chassis_width"    value="0.15"/>
+  <xacro:property name="chassis_height"   value="0.03"/>
+  <!-- Wheel dimensions -->
+  <xacro:property name="wheel_radius"     value="0.0325"/>
+  <xacro:property name="wheel_width"      value="0.025"/>
+  <xacro:property name="wheel_separation" value="0.176"/>
+  <!-- Caster ball radius & chassis height offset -->
+  <xacro:property name="caster_radius"    value="0.00625"/>
+  <xacro:property name="chassis_z"        value="${wheel_radius}"/>
+  <!-- Battery pack dimensions & layout -->
+  <xacro:property name="bat_l"        value="0.055"/>
+  <xacro:property name="bat_w"        value="0.030"/>
+  <xacro:property name="bat_h"        value="0.012"/>
+  <xacro:property name="bat_gap"      value="0.005"/>
+  <xacro:property name="bat_pitch"    value="${bat_w + bat_gap}"/>
   <xacro:property name="bat_center_x" value="-0.055"/>
-  <!-- ═══════════════ BASE LINK ═══════════════ -->
+  <!-- Ball-caster housing geometry -->
+  <xacro:property name="cup_outer_r" value="0.009"/>   <!-- outer radius of cup cylinder -->
+  <xacro:property name="cup_wall_t"  value="0.0015"/>  <!-- wall thickness -->
+  <xacro:property name="cup_h"       value="0.010"/>   <!-- cup body height -->
+  <xacro:property name="cup_top_h"   value="0.003"/>   <!-- top plate height -->
+  <!-- Caster fork ears -->
+  <xacro:property name="ear_w"    value="0.006"/>   <!-- ear width (x) -->
+  <xacro:property name="ear_h"    value="0.008"/>   <!-- ear height (z) -->
+  <xacro:property name="ear_t"    value="0.006"/>   <!-- ear thickness (y) -->
+  <xacro:property name="ear_span" value="0.011"/>   <!-- half-span between ears -->
+  <!-- Caster pivot bolt -->
+  <xacro:property name="pbolt_r" value="0.0025"/>
+  <!-- ════════════════════════════════════════════════════════
+       BASE LINK
+       ════════════════════════════════════════════════════════ -->
   <link name="base_link">
     <inertial>
       <mass value="0.001"/>
-      <inertia ixx="0.000001" ixy="0" ixz="0" iyy="0.000001" iyz="0" izz="0.000001"/>
+      <inertia ixx="0.000001" ixy="0" ixz="0"
+                               iyy="0.000001" iyz="0"
+                                              izz="0.000001"/>
     </inertial>
   </link>
   <joint name="chassis_joint" type="fixed">
     <parent link="base_link"/>
-    <child link="chassis"/>
+    <child  link="chassis"/>
     <origin xyz="0 0 ${chassis_z}" rpy="0 0 0"/>
   </joint>
-  <!-- ═══════════════ CHASSIS ═══════════════ -->
+  <!-- ════════════════════════════════════════════════════════
+       CHASSIS
+       ════════════════════════════════════════════════════════ -->
   <link name="chassis">
     <visual>
@@ -47,8 +71,12 @@
     <inertial>
       <mass value="0.35"/>
-      <inertia ixx="0.000679" ixy="0" ixz="0" iyy="0.001180" iyz="0" izz="0.001639"/>
-    </inertial>
-  </link>
-  <!-- ═══════════════ LEFT WHEEL ═══════════════ -->
+      <inertia ixx="0.000679" ixy="0" ixz="0"
+                               iyy="0.001180" iyz="0"
+                                              izz="0.001639"/>
+    </inertial>
+  </link>
+  <!-- ════════════════════════════════════════════════════════
+       LEFT WHEEL
+       ════════════════════════════════════════════════════════ -->
   <link name="left_wheel">
     <visual>
@@ -69,13 +97,17 @@
     <inertial>
       <mass value="0.06"/>
-      <inertia ixx="0.0000237" ixy="0" ixz="0" iyy="0.0000237" iyz="0" izz="0.0000317"/>
+      <inertia ixx="0.0000237" ixy="0" ixz="0"
+                                iyy="0.0000237" iyz="0"
+                                               izz="0.0000317"/>
     </inertial>
   </link>
   <joint name="left_wheel_joint" type="continuous">
     <parent link="chassis"/>
-    <child link="left_wheel"/>
-    <origin xyz="${-(chassis_length/2 - 0.03)} ${wheel_separation/2} 0" rpy="${-pi/2} 0 0"/>
+    <child  link="left_wheel"/>
+    <origin xyz="${-(chassis_length/2 - 0.03)} ${wheel_separation/2} 0"
+            rpy="${-pi/2} 0 0"/>
     <axis xyz="0 0 1"/>
   </joint>
+  <!-- Left wheel hub (decorative) -->
   <link name="left_wheel_hub">
     <visual>
@@ -90,13 +122,17 @@
     <inertial>
       <mass value="0.005"/>
-      <inertia ixx="0.000001" ixy="0" ixz="0" iyy="0.000001" iyz="0" izz="0.000001"/>
+      <inertia ixx="0.000001" ixy="0" ixz="0"
+                               iyy="0.000001" iyz="0"
+                                              izz="0.000001"/>
     </inertial>
   </link>
   <joint name="left_wheel_hub_joint" type="fixed">
     <parent link="left_wheel"/>
-    <child link="left_wheel_hub"/>
+    <child  link="left_wheel_hub"/>
     <origin xyz="0 0 0" rpy="0 0 0"/>
   </joint>
-  <!-- ═══════════════ RIGHT WHEEL ═══════════════ -->
+  <!-- ════════════════════════════════════════════════════════
+       RIGHT WHEEL
+       ════════════════════════════════════════════════════════ -->
   <link name="right_wheel">
     <visual>
@@ -117,13 +153,17 @@
     <inertial>
       <mass value="0.06"/>
-      <inertia ixx="0.0000237" ixy="0" ixz="0" iyy="0.0000237" iyz="0" izz="0.0000317"/>
+      <inertia ixx="0.0000237" ixy="0" ixz="0"
+                                iyy="0.0000237" iyz="0"
+                                               izz="0.0000317"/>
     </inertial>
   </link>
   <joint name="right_wheel_joint" type="continuous">
     <parent link="chassis"/>
-    <child link="right_wheel"/>
-    <origin xyz="${-(chassis_length/2 - 0.03)} ${-wheel_separation/2} 0" rpy="${-pi/2} 0 0"/>
+    <child  link="right_wheel"/>
+    <origin xyz="${-(chassis_length/2 - 0.03)} ${-wheel_separation/2} 0"
+            rpy="${-pi/2} 0 0"/>
     <axis xyz="0 0 1"/>
   </joint>
+  <!-- Right wheel hub (decorative) -->
   <link name="right_wheel_hub">
     <visual>
@@ -138,13 +178,177 @@
     <inertial>
       <mass value="0.005"/>
-      <inertia ixx="0.000001" ixy="0" ixz="0" iyy="0.000001" iyz="0" izz="0.000001"/>
+      <inertia ixx="0.000001" ixy="0" ixz="0"
+                               iyy="0.000001" iyz="0"
+                                              izz="0.000001"/>
     </inertial>
   </link>
   <joint name="right_wheel_hub_joint" type="fixed">
     <parent link="right_wheel"/>
-    <child link="right_wheel_hub"/>
+    <child  link="right_wheel_hub"/>
     <origin xyz="0 0 0" rpy="0 0 0"/>
   </joint>
-  <!-- ═══════════════ CASTER FRONT ═══════════════ -->
+  <!-- ════════════════════════════════════════════════════════
+       BALL CASTER — additional local properties
+       ════════════════════════════════════════════════════════ -->
+  <xacro:property name="cup_outer_r" value="0.0090"/>   <!-- overrides global -->
+  <xacro:property name="cup_inner_r" value="0.0075"/>
+  <xacro:property name="cup_h"       value="0.0050"/>   <!-- overrides global -->
+  <xacro:property name="cup_top_h"   value="0.0020"/>   <!-- overrides global -->
+  <xacro:property name="cup_embed"   value="0.0020"/>
+  <xacro:property name="caster_top_z"
+    value="${-(caster_radius - wheel_radius) - (cup_top_h/2 + cup_h + caster_radius - cup_embed)}"/>
+  <xacro:property name="ear_w"      value="0.0050"/>    <!-- overrides global -->
+  <xacro:property name="ear_span_y" value="0.0110"/>
+  <xacro:property name="ear_h"      value="0.0060"/>    <!-- overrides global -->
+  <xacro:property name="ear_t"      value="0.0040"/>    <!-- overrides global -->
+  <xacro:property name="pbolt_r"    value="0.0022"/>    <!-- overrides global -->
+  <!-- ── Caster: top mounting plate ── -->
+  <link name="caster_housing_top">
+    <visual>
+      <origin xyz="0 0 0" rpy="0 0 0"/>
+      <geometry>
+        <box size="0.016 0.022 ${cup_top_h}"/>
+      </geometry>
+      <material name="caster_housing_white">
+        <color rgba="0.92 0.90 0.85 1"/>
+      </material>
+    </visual>
+    <collision>
+      <geometry>
+        <box size="0.016 0.022 ${cup_top_h}"/>
+      </geometry>
+    </collision>
+    <inertial>
+      <mass value="0.003"/>
+      <inertia ixx="0.0000015" ixy="0" ixz="0"
+                                iyy="0.0000024" iyz="0"
+                                               izz="0.0000038"/>
+    </inertial>
+  </link>
+  <joint name="caster_housing_top_joint" type="fixed">
+    <parent link="chassis"/>
+    <child  link="caster_housing_top"/>
+    <origin xyz="${chassis_length/2 - 0.020} 0 ${-(chassis_height/2 + cup_top_h/2)}"
+            rpy="0 0 0"/>
+  </joint>
+  <!-- ── Caster: cylindrical cup body ── -->
+  <link name="caster_cup_body">
+    <visual>
+      <origin xyz="0 0 0" rpy="0 0 0"/>
+      <geometry>
+        <cylinder radius="${cup_outer_r}" length="${cup_h}"/>
+      </geometry>
+      <material name="caster_cup_white">
+        <color rgba="0.90 0.88 0.83 1"/>
+      </material>
+    </visual>
+    <collision>
+      <geometry>
+        <cylinder radius="${cup_outer_r}" length="${cup_h}"/>
+      </geometry>
+    </collision>
+    <inertial>
+      <mass value="0.005"/>
+      <inertia ixx="0.0000030" ixy="0" ixz="0"
+                                iyy="0.0000030" iyz="0"
+                                               izz="0.0000036"/>
+    </inertial>
+  </link>
+  <joint name="caster_cup_body_joint" type="fixed">
+    <parent link="caster_housing_top"/>
+    <child  link="caster_cup_body"/>
+    <origin xyz="0 0 ${-(cup_top_h/2 + cup_h/2)}" rpy="0 0 0"/>
+  </joint>
+  <!-- ── Caster: fork ears (left & right) ── -->
+  <link name="caster_ear_left">
+    <visual>
+      <origin xyz="0 0 0" rpy="0 0 0"/>
+      <geometry>
+        <box size="${ear_w} ${ear_t} ${ear_h}"/>
+      </geometry>
+      <material name="caster_ear_white_l">
+        <color rgba="0.90 0.88 0.83 1"/>
+      </material>
+    </visual>
+    <inertial>
+      <mass value="0.002"/>
+      <inertia ixx="0.0000010" ixy="0" ixz="0"
+                                iyy="0.0000008" iyz="0"
+                                               izz="0.0000005"/>
+    </inertial>
+  </link>
+  <joint name="caster_ear_left_joint" type="fixed">
+    <parent link="caster_cup_body"/>
+    <child  link="caster_ear_left"/>
+    <origin xyz="0 ${cup_outer_r + ear_t/2} ${cup_h/2 - ear_h/2}" rpy="0 0 0"/>
+  </joint>
+  <link name="caster_ear_right">
+    <visual>
+      <origin xyz="0 0 0" rpy="0 0 0"/>
+      <geometry>
+        <box size="${ear_w} ${ear_t} ${ear_h}"/>
+      </geometry>
+      <material name="caster_ear_white_r">
+        <color rgba="0.90 0.88 0.83 1"/>
+      </material>
+    </visual>
+    <inertial>
+      <mass value="0.002"/>
+      <inertia ixx="0.0000010" ixy="0" ixz="0"
+                                iyy="0.0000008" iyz="0"
+                                               izz="0.0000005"/>
+    </inertial>
+  </link>
+  <joint name="caster_ear_right_joint" type="fixed">
+    <parent link="caster_cup_body"/>
+    <child  link="caster_ear_right"/>
+    <origin xyz="0 ${-(cup_outer_r + ear_t/2)} ${cup_h/2 - ear_h/2}" rpy="0 0 0"/>
+  </joint>
+  <!-- ── Caster: pivot bolts ── -->
+  <link name="caster_pivot_bolt_left">
+    <visual>
+      <origin xyz="0 0 0" rpy="0 0 0"/>
+      <geometry>
+        <sphere radius="${pbolt_r}"/>
+      </geometry>
+      <material name="pivot_bolt_dark_l">
+        <color rgba="0.12 0.12 0.12 1"/>
+      </material>
+    </visual>
+    <inertial>
+      <mass value="0.001"/>
+      <inertia ixx="0.0000001" ixy="0" ixz="0"
+                                iyy="0.0000001" iyz="0"
+                                               izz="0.0000001"/>
+    </inertial>
+  </link>
+  <joint name="caster_pivot_bolt_left_joint" type="fixed">
+    <parent link="caster_ear_left"/>
+    <child  link="caster_pivot_bolt_left"/>
+    <origin xyz="0 ${ear_t/2 + pbolt_r * 0.3} 0" rpy="0 0 0"/>
+  </joint>
+  <link name="caster_pivot_bolt_right">
+    <visual>
+      <origin xyz="0 0 0" rpy="0 0 0"/>
+      <geometry>
+        <sphere radius="${pbolt_r}"/>
+      </geometry>
+      <material name="pivot_bolt_dark_r">
+        <color rgba="0.12 0.12 0.12 1"/>
+      </material>
+    </visual>
+    <inertial>
+      <mass value="0.001"/>
+      <inertia ixx="0.0000001" ixy="0" ixz="0"
+                                iyy="0.0000001" iyz="0"
+                                               izz="0.0000001"/>
+    </inertial>
+  </link>
+  <joint name="caster_pivot_bolt_right_joint" type="fixed">
+    <parent link="caster_ear_right"/>
+    <child  link="caster_pivot_bolt_right"/>
+    <origin xyz="0 ${-(ear_t/2 + pbolt_r * 0.3)} 0" rpy="0 0 0"/>
+  </joint>
+  <!-- ── Caster: rolling ball ── -->
   <link name="caster_front">
     <visual>
@@ -153,23 +357,55 @@
         <sphere radius="${caster_radius}"/>
       </geometry>
-      <material name="caster_silver">
-        <color rgba="0.72 0.72 0.74 1"/>
+      <material name="caster_ball_dark">
+        <color rgba="0.15 0.15 0.16 1"/>
       </material>
     </visual>
     <collision>
-      <geometry><sphere radius="${caster_radius}"/></geometry>
+      <geometry>
+        <sphere radius="${caster_radius}"/>
+      </geometry>
     </collision>
     <inertial>
-      <mass value="0.01"/>
-      <inertia ixx="0.00000058" ixy="0" ixz="0" iyy="0.00000058" iyz="0" izz="0.00000058"/>
+      <mass value="0.010"/>
+      <inertia ixx="0.00000058" ixy="0" ixz="0"
+                                 iyy="0.00000058" iyz="0"
+                                                  izz="0.00000058"/>
     </inertial>
   </link>
   <joint name="caster_front_joint" type="fixed">
-    <parent link="chassis"/>
-    <child link="caster_front"/>
-    <origin xyz="${chassis_length/2 - 0.02} 0 ${caster_radius - wheel_radius}" rpy="0 0 0"/>
-  </joint>
-  <!-- ═══════════════ BATTERY UNIT ═══════════════ -->
+    <parent link="caster_housing_top"/>
+    <child  link="caster_front"/>
+    <origin xyz="0 0 -0.0103" rpy="0 0 0"/>
+  </joint>
+  <!-- ── Caster: specular highlight (decorative) ── -->
+  <link name="caster_ball_shine">
+    <visual>
+      <origin xyz="0 0 0" rpy="0 0 0"/>
+      <geometry>
+        <sphere radius="${caster_radius * 0.25}"/>
+      </geometry>
+      <material name="caster_ball_spec">
+        <color rgba="0.60 0.60 0.62 0.55"/>
+      </material>
+    </visual>
+    <inertial>
+      <mass value="0.0001"/>
+      <inertia ixx="0.0000001" ixy="0" ixz="0"
+                                iyy="0.0000001" iyz="0"
+                                               izz="0.0000001"/>
+    </inertial>
+  </link>
+  <joint name="caster_ball_shine_joint" type="fixed">
+    <parent link="caster_front"/>
+    <child  link="caster_ball_shine"/>
+    <origin xyz="${-caster_radius * 0.3} 0 ${caster_radius * 0.65}" rpy="0 0 0"/>
+  </joint>
+  <!-- ════════════════════════════════════════════════════════
+       BATTERY UNIT — xacro macro
+       Params : side      → name suffix (e.g. "single")
+                x_offset  → x position on chassis
+       ════════════════════════════════════════════════════════ -->
   <xacro:macro name="battery_unit" params="side x_offset">
+    <!-- Main cell body -->
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